Commit message: Mon robot humanoide complet avec bras et jambes

File: urdf/humanoid.urdf (robot description, URDF)
Before this commit: robot humanoid, 1 links, 0 joints
Links:
- added link head; visual sphere radius=0.1
- added link left_arm; visual cylinder length=0.3 radius=0.04
- added link left_leg; visual cylinder length=0.4 radius=0.05
- added link right_arm; visual cylinder length=0.3 radius=0.04
- added link right_leg; visual cylinder length=0.4 radius=0.05
- link base_link: geometry visual box size=0.2 0.3 0.4
Joints:
- added joint left_hip_joint: type fixed, parent base_link, child left_leg, origin xyz=0 0.1 -0.4 rpy=0 0 0
- added joint left_shoulder_joint: type fixed, parent base_link, child left_arm, origin xyz=0 0.2 0.1 rpy=0 0 0
- added joint neck_joint: type fixed, parent base_link, child head, origin xyz=0 0 0.3 rpy=0 0 0
- added joint right_hip_joint: type fixed, parent base_link, child right_leg, origin xyz=0 -0.1 -0.4 rpy=0 0 0
- added joint right_shoulder_joint: type fixed, parent base_link, child right_arm, origin xyz=0 -0.2 0.1 rpy=0 0 0

Commit message: Correction du positionnement des membres de l'iCub

File: urdf/humanoid.urdf (robot description, URDF)
Before this commit: robot humanoid_robot, 6 links, 5 joints
Links:
- removed link left_arm
- removed link left_leg
- removed link right_arm
- removed link right_leg
- added link l_arm; visual mesh filename=package://humanoid_robot/meshes/l_upper_arm.dae scale=0.001 0.001 0.001
- added link l_foot; visual mesh filename=package://humanoid_robot/meshes/l_foot.dae scale=0.001 0.001 0.001
- added link l_forearm; visual box size=0.03 0.03 0.15
- added link l_hand; visual box size=0.04 0.02 0.08
- added link l_leg; visual mesh filename=package://humanoid_robot/meshes/l_upper_leg.dae scale=0.001 0.001 0.001
- added link l_lower_leg; visual mesh filename=package://humanoid_robot/meshes/l_lower_leg.dae scale=0.001 0.001 0.001
- added link r_arm; visual mesh filename=package://humanoid_robot/meshes/r_upper_arm.dae scale=0.001 0.001 0.001
- added link r_foot; visual mesh filename=package://humanoid_robot/meshes/r_foot.dae scale=0.001 0.001 0.001
- added link r_forearm; visual box size=0.03 0.03 0.15
- added link r_hand; visual box size=0.04 0.02 0.08
- added link r_leg; visual mesh filename=package://humanoid_robot/meshes/r_upper_leg.dae scale=0.001 0.001 0.001
- added link r_lower_leg; visual mesh filename=package://humanoid_robot/meshes/r_lower_leg.dae scale=0.001 0.001 0.001
- link base_link: geometry visual mesh filename=package://humanoid_robot/meshes/chest.dae scale=0.001 0.001 0.001
- link head: geometry visual mesh filename=package://humanoid_robot/meshes/head.dae scale=0.001 0.001 0.001
Joints:
- removed joint left_hip_joint
- removed joint left_shoulder_joint
- removed joint neck_joint
- removed joint right_hip_joint
- removed joint right_shoulder_joint
- added joint head_joint: type fixed, parent base_link, child head, origin xyz=0 0 0.18
- added joint l_arm_j: type fixed, parent base_link, child l_arm, origin xyz=0 0.12 0.12
- added joint l_foot_j: type fixed, parent l_lower_leg, child l_foot, origin xyz=0 0 -0.2
- added joint l_forearm_j: type fixed, parent l_arm, child l_forearm, origin xyz=0 0 -0.15
- added joint l_hand_j: type fixed, parent l_forearm, child l_hand, origin xyz=0 0 -0.12
- added joint l_leg_j: type fixed, parent base_link, child l_leg, origin xyz=0 0.05 -0.2
- added joint l_lower_leg_j: type fixed, parent l_leg, child l_lower_leg, origin xyz=0 0 -0.25
- added joint r_arm_j: type fixed, parent base_link, child r_arm, origin xyz=0 -0.12 0.12
- added joint r_foot_j: type fixed, parent r_lower_leg, child r_foot, origin xyz=0 0 -0.2
- added joint r_forearm_j: type fixed, parent r_arm, child r_forearm, origin xyz=0 0 -0.15
- added joint r_hand_j: type fixed, parent r_forearm, child r_hand, origin xyz=0 0 -0.12
- added joint r_leg_j: type fixed, parent base_link, child r_leg, origin xyz=0 -0.05 -0.2
- added joint r_lower_leg_j: type fixed, parent r_leg, child r_lower_leg, origin xyz=0 0 -0.25

Commit message: Correction du positionnement des membres de l'iCub

File: urdf/humanoid.urdf (robot description, URDF)
Before this commit: robot iCub, 14 links, 13 joints
Joints:
- joint head_joint: origin xyz=0 0 0.18 -> xyz=0 0 0.16
- joint l_arm_j: origin xyz=0 0.12 0.12 -> xyz=0 0.06 0.10
- joint l_foot_j: origin xyz=0 0 -0.2 -> xyz=0 0 -0.15
- joint l_forearm_j: origin xyz=0 0 -0.15 -> xyz=0 0 -0.10
- joint l_hand_j: origin xyz=0 0 -0.12 -> xyz=0 0 -0.10
- joint l_leg_j: origin xyz=0 0.05 -0.2 -> xyz=0 0.04 -0.05
- joint l_lower_leg_j: origin xyz=0 0 -0.25 -> xyz=0 0 -0.18
- joint r_arm_j: origin xyz=0 -0.12 0.12 -> xyz=0 -0.06 0.10
- joint r_foot_j: origin xyz=0 0 -0.2 -> xyz=0 0 -0.15
- joint r_forearm_j: origin xyz=0 0 -0.15 -> xyz=0 0 -0.10
- joint r_hand_j: origin xyz=0 0 -0.12 -> xyz=0 0 -0.10
- joint r_leg_j: origin xyz=0 -0.05 -0.2 -> xyz=0 -0.04 -0.05
- joint r_lower_leg_j: origin xyz=0 0 -0.25 -> xyz=0 0 -0.18

Commit message: Envoi du projet Robot Humanoïde : Conception et Simulation

File: urdf/humanoid.urdf (robot description, URDF)
Before this commit: robot iCub, 56 links, 55 joints
Links:
- removed link bb_chest_link
- removed link head_imu_frame
- removed link l_arm
- removed link l_arm_back_cover
- removed link l_arm_cover
- removed link l_calf_cover
- removed link l_hip_visual
- removed link l_leg
- removed link l_shoulder
- removed link l_thigh_cover
- removed link l_wrist
- removed link lap_belt_link
- removed link neck
- removed link r_arm
- removed link r_arm_back_cover
- removed link r_arm_cover
- removed link r_calf_cover
- removed link r_hip_visual
- removed link r_leg
- removed link r_shoulder
- removed link r_thigh_cover
- removed link r_wrist
- added link chest; visual mesh filename=package://humanoid_robot/meshes/chest.dae scale=0.001 0.001 0.001
- added link l_ankle_1; visual mesh filename=package://humanoid_robot/meshes/l_ankle_1.dae scale=0.001 0.001 0.001
- added link l_ankle_2; visual mesh filename=package://humanoid_robot/meshes/l_ankle_2.dae scale=0.001 0.001 0.001
- added link l_elbow_1; visual mesh filename=package://humanoid_robot/meshes/l_elbow_1.dae scale=0.001 0.001 0.001
- added link l_hip_1; visual mesh filename=package://humanoid_robot/meshes/l_hip_1.dae scale=0.001 0.001 0.001
- added link l_hip_2; visual mesh filename=package://humanoid_robot/meshes/l_hip_2.dae scale=0.001 0.001 0.001
- added link l_hip_3; visual mesh filename=package://humanoid_robot/meshes/l_hip_3.dae scale=0.001 0.001 0.001
- added link l_shoulder_1; visual mesh filename=package://humanoid_robot/meshes/l_shoulder_1.dae scale=0.001 0.001 0.001
- added link l_shoulder_2; visual mesh filename=package://humanoid_robot/meshes/l_shoulder_2.dae scale=0.001 0.001 0.001
- added link l_shoulder_3; visual mesh filename=package://humanoid_robot/meshes/l_shoulder_3.dae scale=0.001 0.001 0.001
- added link l_sole
- added link l_upper_arm; visual mesh filename=package://humanoid_robot/meshes/l_upper_arm.dae scale=0.001 0.001 0.001
- added link l_upper_leg; visual mesh filename=package://humanoid_robot/meshes/l_upper_leg.dae scale=0.001 0.001 0.001
- added link l_wrist_1; visual mesh filename=package://humanoid_robot/meshes/l_wrist_1.dae scale=0.001 0.001 0.001
- added link neck_1; visual mesh filename=package://humanoid_robot/meshes/neck_1.dae scale=0.001 0.001 0.001
- added link r_ankle_1; visual mesh filename=package://humanoid_robot/meshes/r_ankle_1.dae scale=0.001 0.001 0.001
- added link r_ankle_2; visual mesh filename=package://humanoid_robot/meshes/r_ankle_2.dae scale=0.001 0.001 0.001
- added link r_elbow_1; visual mesh filename=package://humanoid_robot/meshes/r_elbow_1.dae scale=0.001 0.001 0.001
- added link r_hip_1; visual mesh filename=package://humanoid_robot/meshes/r_hip_1.dae scale=0.001 0.001 0.001
- added link r_hip_2; visual mesh filename=package://humanoid_robot/meshes/r_hip_2.dae scale=0.001 0.001 0.001
- added link r_hip_3; visual mesh filename=package://humanoid_robot/meshes/r_hip_3.dae scale=0.001 0.001 0.001
- added link r_shoulder_1; visual mesh filename=package://humanoid_robot/meshes/r_shoulder_1.dae scale=0.001 0.001 0.001
- added link r_shoulder_2; visual mesh filename=package://humanoid_robot/meshes/r_shoulder_2.dae scale=0.001 0.001 0.001
- added link r_shoulder_3; visual mesh filename=package://humanoid_robot/meshes/r_shoulder_3.dae scale=0.001 0.001 0.001
- added link r_sole
- added link r_upper_arm; visual mesh filename=package://humanoid_robot/meshes/r_upper_arm.dae scale=0.001 0.001 0.001
- added link r_upper_leg; visual mesh filename=package://humanoid_robot/meshes/r_upper_leg.dae scale=0.001 0.001 0.001
- added link r_wrist_1; visual mesh filename=package://humanoid_robot/meshes/r_wrist_1.dae scale=0.001 0.001 0.001
- added link torso_1; visual mesh filename=package://humanoid_robot/meshes/torso_1.dae scale=0.001 0.001 0.001
- added link torso_2; visual mesh filename=package://humanoid_robot/meshes/torso_2.dae scale=0.001 0.001 0.001
- link base_link: mass 3.0 -> None; geometry 
- link head: mass 0.8 -> None; geometry visual mesh filename=package://humanoid_robot/meshes/head.dae scale=0.001 0.001 0.001
- link l_eye: mass 0.02 -> None
- link l_foot: mass 0.3 -> None; geometry visual mesh filename=package://humanoid_robot/meshes/l_foot.dae scale=0.001 0.001 0.001
- link l_forearm: mass 0.35 -> None; geometry visual mesh filename=package://humanoid_robot/meshes/l_forearm.dae scale=0.001 0.001 0.001
- link l_hand: mass 0.18 -> None; geometry visual mesh filename=package://humanoid_robot/meshes/l_hand.dae scale=0.001 0.001 0.001
- link l_index_distal: mass 0.005 -> None
- link l_index_proximal: mass 0.008 -> None
- link l_lower_leg: mass 0.6 -> None; geometry visual mesh filename=package://humanoid_robot/meshes/l_lower_leg.dae scale=0.001 0.001 0.001
- link l_middle_distal: mass 0.005 -> None
- link l_middle_proximal: mass 0.008 -> None
- link l_pinky_distal: mass 0.003 -> None
- link l_pinky_proximal: mass 0.005 -> None
- link l_ring_distal: mass 0.004 -> None
- link l_ring_proximal: mass 0.007 -> None
- link l_thumb_distal: mass 0.007 -> None
- link l_thumb_proximal: mass 0.010 -> None
- link r_eye: mass 0.02 -> None
- link r_foot: mass 0.3 -> None; geometry visual mesh filename=package://humanoid_robot/meshes/r_foot.dae scale=0.001 0.001 0.001
- link r_forearm: mass 0.35 -> None; geometry visual mesh filename=package://humanoid_robot/meshes/r_forearm.dae scale=0.001 0.001 0.001
- link r_hand: mass 0.18 -> None; geometry visual mesh filename=package://humanoid_robot/meshes/r_hand.dae scale=0.001 0.001 0.001
- link r_index_distal: mass 0.005 -> None
- link r_index_proximal: mass 0.008 -> None
- link r_lower_leg: mass 0.6 -> None; geometry visual mesh filename=package://humanoid_robot/meshes/r_lower_leg.dae scale=0.001 0.001 0.001
- link r_middle_distal: mass 0.005 -> None
- link r_middle_proximal: mass 0.008 -> None
- link r_pinky_distal: mass 0.003 -> None
- link r_pinky_proximal: mass 0.005 -> None
- link r_ring_distal: mass 0.004 -> None
- link r_ring_proximal: mass 0.007 -> None
- link r_thumb_distal: mass 0.007 -> None
- link r_thumb_proximal: mass 0.010 -> None
- link root_link: mass 1.5 -> None; geometry visual mesh filename=package://humanoid_robot/meshes/root.dae scale=0.001 0.001 0.001
Joints:
- removed joint bb_chest_joint
- removed joint head_imu_joint
- removed joint head_joint
- removed joint l_ankle_joint
- removed joint l_arm_back_cover_joint
- removed joint l_arm_cover_joint
- removed joint l_arm_j
- removed joint l_calf_cover_joint
- removed joint l_forearm_j
- removed joint l_hand_joint
- removed joint l_hip_v_joint
- removed joint l_knee_joint
- removed joint l_leg_j
- removed joint l_shoulder_joint
- removed joint l_thigh_cover_joint
- removed joint l_wrist_joint
- removed joint lap_belt_joint
- removed joint neck_2_joint
- removed joint neck_joint
- removed joint r_ankle_joint
- removed joint r_arm_back_cover_joint
- removed joint r_arm_cover_joint
- removed joint r_arm_j
- removed joint r_calf_cover_joint
- removed joint r_forearm_j
- removed joint r_hand_joint
- removed joint r_hip_v_joint
- removed joint r_knee_joint
- removed joint r_leg_j
- removed joint r_shoulder_joint
- removed joint r_thigh_cover_joint
- removed joint r_wrist_joint
- removed joint root_joint
- added joint base_link_fixed_joint: type fixed, parent root_link, child base_link, origin xyz=0 0 0 rpy=0 0 0
- added joint l_ankle_pitch: type revolute, parent l_lower_leg, child l_ankle_1, origin xyz=0 0 -0.200500 rpy=0 0 0, axis 0 1 0, limit lower=-0.610865 upper=0.610865 effort=37.0 velocity=7.64
- added joint l_ankle_roll: type revolute, parent l_ankle_1, child l_ankle_2, origin xyz=0 0 0 rpy=0 0 0, axis 1 0 0, limit lower=-0.436332 upper=0.436332 effort=37.0 velocity=7.64
- added joint l_arm_ft_sensor: type fixed, parent l_shoulder_3, child l_upper_arm, origin xyz=0.050930 0 0.029176 rpy=0 -1.308997 3.141593
- added joint l_elbow: type revolute, parent l_upper_arm, child l_elbow_1, origin xyz=0 0.034000 0.079260 rpy=0 -1.308997 -3.141593, axis 0 -1 0, limit lower=0.261799 upper=1.850049 effort=50000 velocity=50000
- added joint l_foot_ft_sensor: type fixed, parent l_ankle_2, child l_foot, origin xyz=-0.003500 0 -0.060500 rpy=3.141593 0 0
- added joint l_hip_pitch: type revolute, parent root_link, child l_hip_1, origin xyz=0.006452 -0.026000 -0.119913 rpy=0 0 -3.141593, axis 0 -1 0, limit lower=-0.785398 upper=2.338741 effort=55.5 velocity=5.1
- added joint l_hip_roll: type revolute, parent l_hip_1, child l_hip_2, origin xyz=0 0.044100 0 rpy=0 0 0, axis 1 0 0, limit lower=-0.349066 upper=2.094395 effort=37.0 velocity=7.64
- added joint l_hip_yaw: type revolute, parent l_hip_3, child l_upper_leg, origin xyz=0 0 0.014400 rpy=-3.141593 0 0, axis 0 0 1, limit lower=-1.396263 upper=1.396263 effort=37.0 velocity=7.64
- added joint l_knee: type revolute, parent l_upper_leg, child l_lower_leg, origin xyz=0 0 -0.145825 rpy=0 0 0, axis 0 -1 0, limit lower=-2.164208 upper=0.069813 effort=37.0 velocity=7.64
- added joint l_leg_ft_sensor: type fixed, parent l_hip_2, child l_hip_3, origin xyz=-0.000830 0.000075 -0.074300 rpy=3.141593 0 0
- added joint l_shoulder_pitch: type revolute, parent chest, child l_shoulder_1, origin xyz=0.120016 0.092800 0.007969 rpy=0 0 0, axis 0.965926 0 0.258819, limit lower=-1.666789 upper=0.174533 effort=50000 velocity=50000
- added joint l_shoulder_roll: type revolute, parent l_shoulder_1, child l_shoulder_2, origin xyz=-0.013671 0 0.008520 rpy=0.270597 0.252680 -1.501557, axis -0.258819 0 0.965926, limit lower=0.0 upper=2.806489 effort=50000 velocity=50000
- added joint l_shoulder_yaw: type revolute, parent l_shoulder_2, child l_shoulder_3, origin xyz=0.025314 0 -0.005401 rpy=-0.252690 -0.008519 -0.067040, axis 0.965926 0 0.258819, limit lower=-0.645772 upper=1.396263 effort=50000 velocity=50000
- added joint l_sole_fixed_joint: type fixed, parent l_foot, child l_sole, origin xyz=0.003500 0 0.004000 rpy=-3.141593 0 0
- added joint l_wrist_pitch: type revolute, parent l_forearm, child l_wrist_1, origin xyz=0.103428 0.000007 0.025487 rpy=0 0 0, axis 0.258819 0 -0.965926, limit lower=-1.396263 upper=0.436332 effort=50000 velocity=50000
- added joint l_wrist_prosup: type revolute, parent l_elbow_1, child l_forearm, origin xyz=0.038462 0.034000 -0.005223 rpy=0 0 0, axis 0.965926 0 0.258819, limit lower=-1.047198 upper=1.047198 effort=50000 velocity=50000
- added joint l_wrist_yaw: type revolute, parent l_wrist_1, child l_hand, origin xyz=-0.000634 -0.019500 0.002367 rpy=0 0 0, axis 0 1 0, limit lower=-0.349066 upper=0.436332 effort=50000 velocity=50000
- added joint neck_pitch: type revolute, parent chest, child neck_1, origin xyz=-0.014300 0.172797 0.005312 rpy=0 0 0, axis -1 0 0, limit lower=-0.698132 upper=0.383972 effort=50000 velocity=50000
- added joint neck_roll: type revolute, parent neck_1, child neck_2, origin xyz=0.014300 0.009500 0.020800 rpy=0 0 0, axis 0 0 1, limit lower=-0.349066 upper=0.349066 effort=50000 velocity=50000
- added joint neck_yaw: type revolute, parent neck_2, child head, origin xyz=0 -0.022344 -0.020800 rpy=0 0 0, axis 0 1 0, limit lower=-0.872665 upper=0.872665 effort=50000 velocity=50000
- added joint r_ankle_pitch: type revolute, parent r_lower_leg, child r_ankle_1, origin xyz=0 0 -0.200500 rpy=0 0 0, axis 0 1 0, limit lower=-0.610865 upper=0.610865 effort=37.0 velocity=7.64
- added joint r_ankle_roll: type revolute, parent r_ankle_1, child r_ankle_2, origin xyz=0 0 0 rpy=0 0 0, axis -1 0 0, limit lower=-0.436332 upper=0.436332 effort=37.0 velocity=7.64
- added joint r_arm_ft_sensor: type fixed, parent r_shoulder_3, child r_upper_arm, origin xyz=-0.050897 0 0.029167 rpy=0 -1.308997 0
- added joint r_elbow: type revolute, parent r_upper_arm, child r_elbow_1, origin xyz=0 -0.022500 0.079260 rpy=0 1.308997 0, axis 0 1 0, limit lower=0.261799 upper=1.850049 effort=50000 velocity=50000
- added joint r_foot_ft_sensor: type fixed, parent r_ankle_2, child r_foot, origin xyz=-0.003500 0 -0.060500 rpy=3.141593 0 0
- added joint r_hip_pitch: type revolute, parent root_link, child r_hip_1, origin xyz=0.006452 0.026000 -0.119913 rpy=0 0 -3.141593, axis 0 -1 0, limit lower=-0.785398 upper=2.338741 effort=55.5 velocity=5.1
- added joint r_hip_roll: type revolute, parent r_hip_1, child r_hip_2, origin xyz=0 -0.044100 0 rpy=0 0 0, axis -1 0 0, limit lower=-0.349066 upper=2.094395 effort=37.0 velocity=7.64
- added joint r_hip_yaw: type revolute, parent r_hip_3, child r_upper_leg, origin xyz=0 0 0.014400 rpy=-3.141593 0 0, axis 0 0 -1, limit lower=-1.396263 upper=1.396263 effort=37.0 velocity=7.64
- added joint r_knee: type revolute, parent r_upper_leg, child r_lower_leg, origin xyz=0 0 -0.145825 rpy=0 0 0, axis 0 -1 0, limit lower=-2.164208 upper=0.069813 effort=37.0 velocity=7.64
- added joint r_leg_ft_sensor: type fixed, parent r_hip_2, child r_hip_3, origin xyz=-0.000936 0.000014 -0.074300 rpy=3.141593 0 0
- added joint r_shoulder_pitch: type revolute, parent chest, child r_shoulder_1, origin xyz=-0.120016 0.092800 0.007969 rpy=0 -0.523599 3.141593, axis -0.965926 0 0.258819, limit lower=-1.666789 upper=0.174533 effort=50000 velocity=50000
- added joint r_shoulder_roll: type revolute, parent r_shoulder_1, child r_shoulder_2, origin xyz=-0.007580 0 0.014210 rpy=-0.270598 -0.252680 -1.501557, axis -0.258819 0 -0.965926, limit lower=0.0 upper=2.806489 effort=50000 velocity=50000
- added joint r_shoulder_yaw: type revolute, parent r_shoulder_2, child r_shoulder_3, origin xyz=-0.025346 0 -0.005388 rpy=-0.252690 0.008519 0.067040, axis 0.965926 0 -0.258819, limit lower=-0.645772 upper=1.396263 effort=50000 velocity=50000
- added joint r_sole_fixed_joint: type fixed, parent r_foot, child r_sole, origin xyz=0.003500 0 0.004000 rpy=-3.141593 0 0
- added joint r_wrist_pitch: type revolute, parent r_forearm, child r_wrist_1, origin xyz=-0.103505 0.000007 0.025198 rpy=0 0 0, axis 0.258819 0 0.965926, limit lower=-1.396263 upper=0.436332 effort=50000 velocity=50000
- added joint r_wrist_prosup: type revolute, parent r_elbow_1, child r_forearm, origin xyz=-0.038462 0.022500 -0.005223 rpy=0 0 0, axis 0.965926 0 -0.258819, limit lower=-1.047198 upper=1.047198 effort=50000 velocity=50000
- added joint r_wrist_yaw: type revolute, parent r_wrist_1, child r_hand, origin xyz=0.000634 -0.019500 0.002367 rpy=0 0 0, axis 0 -1 0, limit lower=-0.349066 upper=0.436332 effort=50000 velocity=50000
- added joint torso_pitch: type revolute, parent root_link, child torso_1, origin xyz=0 0.027046 0 rpy=1.5707963 0 -1.5707963, axis 1 0 0, limit lower=-0.349066 upper=1.221730 effort=50000 velocity=50000
- added joint torso_roll: type revolute, parent torso_1, child torso_2, origin xyz=0.027046 0.032 -0.057345 rpy=0 0 0, axis 0 0 -1, limit lower=-0.523599 upper=0.523599 effort=50000 velocity=50000
- added joint torso_yaw: type revolute, parent torso_2, child chest, origin xyz=0 0.05 0.062842 rpy=0 0 0, axis 0 -1 0, limit lower=-0.872665 upper=0.872665 effort=50000 velocity=50000
- joint l_eye_joint: origin xyz=0.07 0.033 0.055 -> xyz=0.034 0.082 0.026
- joint r_eye_joint: origin xyz=0.07 -0.033 0.055 -> xyz=-0.034 0.082 0.026

Commit message: Envoi du projet Robot Humanoïde : Conception et Simulation

File: urdf/humanoid.urdf (robot description, URDF)
Before this commit: robot iCub, 64 links, 63 joints
Links:
- link r_ankle_2: geometry 
Joints:
- joint l_index_proximal_j: origin xyz=0.012 0.02 -0.075 -> xyz=0.010 0.010 -0.072
- joint l_middle_proximal_j: origin xyz=0.004 0.02 -0.075 -> xyz=0.003 0.010 -0.074
- joint l_pinky_proximal_j: origin xyz=-0.012 0.018 -0.065 -> xyz=-0.010 0.008 -0.063
- joint l_ring_proximal_j: origin xyz=-0.004 0.02 -0.073 -> xyz=-0.004 0.010 -0.071
- joint l_thumb_proximal_j: origin xyz=0.025 0.005 -0.040 rpy=0 0.5 0 -> xyz=0.020 0.010 -0.042 rpy=0 0.5 0
- joint r_index_proximal_j: origin xyz=-0.012 0.02 -0.075 -> xyz=-0.010 0.010 -0.072
- joint r_middle_proximal_j: origin xyz=-0.004 0.02 -0.075 -> xyz=-0.003 0.010 -0.074
- joint r_pinky_proximal_j: origin xyz=0.012 0.018 -0.065 -> xyz=0.010 0.008 -0.063
- joint r_ring_proximal_j: origin xyz=0.004 0.02 -0.073 -> xyz=0.004 0.010 -0.071
- joint r_thumb_proximal_j: origin xyz=-0.025 0.005 -0.040 rpy=0 0.5 0 -> xyz=-0.020 0.010 -0.042 rpy=0 0.5 0

Commit message: Ajout des photos RViz et mise à jour du README

File: urdf/humanoid.urdf (robot description, URDF)
Before this commit: robot iCub, 64 links, 63 joints
Links:
- link r_ankle_2: geometry visual mesh filename=package://humanoid_robot/meshes/r_ankle_2.dae scale=0.001 0.001 0.001
Joints:
- joint l_index_proximal_j: origin xyz=0.010 0.010 -0.072 -> xyz=0.012 0.02 -0.075
- joint l_middle_proximal_j: origin xyz=0.003 0.010 -0.074 -> xyz=0.004 0.02 -0.075
- joint l_pinky_proximal_j: origin xyz=-0.010 0.008 -0.063 -> xyz=-0.012 0.018 -0.065
- joint l_ring_proximal_j: origin xyz=-0.004 0.010 -0.071 -> xyz=-0.004 0.02 -0.073
- joint l_thumb_proximal_j: origin xyz=0.020 0.010 -0.042 rpy=0 0.5 0 -> xyz=0.025 0.005 -0.040 rpy=0 0.5 0
- joint r_index_proximal_j: origin xyz=-0.010 0.010 -0.072 -> xyz=-0.012 0.02 -0.075
- joint r_middle_proximal_j: origin xyz=-0.003 0.010 -0.074 -> xyz=-0.004 0.02 -0.075
- joint r_pinky_proximal_j: origin xyz=0.010 0.008 -0.063 -> xyz=0.012 0.018 -0.065
- joint r_ring_proximal_j: origin xyz=0.004 0.010 -0.071 -> xyz=0.004 0.02 -0.073
- joint r_thumb_proximal_j: origin xyz=-0.020 0.010 -0.042 rpy=0 0.5 0 -> xyz=-0.025 0.005 -0.040 rpy=0 0.5 0
