Commit message: Amélioration: articulations actives pour les doigts avec 3 phalanges dans humanoid.urdf

File: urdf/humanoid.urdf (robot description, URDF)
Before this commit: robot iCub, 64 links, 63 joints
Links:
- added link l_index_middle, mass 0.05; collision cylinder length=0.030 radius=0.007; visual cylinder length=0.030 radius=0.007
- added link l_middle_middle, mass 0.055; collision cylinder length=0.034 radius=0.007; visual cylinder length=0.034 radius=0.007
- added link l_pinky_middle, mass 0.03; collision cylinder length=0.024 radius=0.005; visual cylinder length=0.024 radius=0.005
- added link l_ring_middle, mass 0.04; collision cylinder length=0.028 radius=0.006; visual cylinder length=0.028 radius=0.006
- added link l_thumb_middle, mass 0.07; collision cylinder length=0.032 radius=0.008; visual cylinder length=0.032 radius=0.008
- added link r_index_middle, mass 0.05; collision cylinder length=0.030 radius=0.007; visual cylinder length=0.030 radius=0.007
- added link r_middle_middle, mass 0.055; collision cylinder length=0.034 radius=0.007; visual cylinder length=0.034 radius=0.007
- added link r_pinky_middle, mass 0.03; collision cylinder length=0.024 radius=0.005; visual cylinder length=0.024 radius=0.005
- added link r_ring_middle, mass 0.04; collision cylinder length=0.028 radius=0.006; visual cylinder length=0.028 radius=0.006
- added link r_thumb_middle, mass 0.07; collision cylinder length=0.032 radius=0.008; visual cylinder length=0.032 radius=0.008
- link chest: mass None -> 1.0; geometry collision sphere radius=0.1; visual mesh filename=package://humanoid_robot/meshes/chest.dae scale=0.001 0.001 0.001
- link head: mass None -> 0.6; geometry collision sphere radius=0.055; visual mesh filename=package://humanoid_robot/meshes/head.dae scale=0.001 0.001 0.001
- link l_ankle_1: mass None -> 0.3; geometry collision sphere radius=0.03; visual mesh filename=package://humanoid_robot/meshes/l_ankle_1.dae scale=0.001 0.001 0.001
- link l_ankle_2: mass None -> 0.25; geometry collision sphere radius=0.028; visual mesh filename=package://humanoid_robot/meshes/l_ankle_2.dae scale=0.001 0.001 0.001
- link l_elbow_1: mass None -> 0.25; geometry collision sphere radius=0.025; visual mesh filename=package://humanoid_robot/meshes/l_elbow_1.dae scale=0.001 0.001 0.001
- link l_eye: mass None -> 0.01
- link l_foot: mass None -> 0.4; geometry collision box size=0.1 0.08 0.02; visual mesh filename=package://humanoid_robot/meshes/l_foot.dae scale=0.001 0.001 0.001
- link l_forearm: mass None -> 0.3; geometry collision cylinder length=0.18 radius=0.02; visual mesh filename=package://humanoid_robot/meshes/l_forearm.dae scale=0.001 0.001 0.001
- link l_hand: mass None -> 0.2; geometry collision sphere radius=0.025; visual mesh filename=package://humanoid_robot/meshes/l_hand.dae scale=0.001 0.001 0.001
- link l_hip_1: mass None -> 0.5; geometry collision sphere radius=0.045; visual mesh filename=package://humanoid_robot/meshes/l_hip_1.dae scale=0.001 0.001 0.001
- link l_hip_2: mass None -> 0.45; geometry collision sphere radius=0.04; visual mesh filename=package://humanoid_robot/meshes/l_hip_2.dae scale=0.001 0.001 0.001
- link l_hip_3: mass None -> 0.35; geometry collision sphere radius=0.035; visual mesh filename=package://humanoid_robot/meshes/l_hip_3.dae scale=0.001 0.001 0.001
- link l_index_distal: mass None -> 0.03; geometry collision cylinder length=0.025 radius=0.006; visual cylinder length=0.025 radius=0.006
- link l_index_proximal: mass None -> 0.08; geometry collision cylinder length=0.040 radius=0.008; visual cylinder length=0.040 radius=0.008
- link l_lower_leg: mass None -> 0.5; geometry collision cylinder length=0.25 radius=0.03; visual mesh filename=package://humanoid_robot/meshes/l_lower_leg.dae scale=0.001 0.001 0.001
- link l_middle_distal: mass None -> 0.035; geometry collision cylinder length=0.028 radius=0.006; visual cylinder length=0.028 radius=0.006
- link l_middle_proximal: mass None -> 0.09; geometry collision cylinder length=0.042 radius=0.008; visual cylinder length=0.042 radius=0.008
- link l_pinky_distal: mass None -> 0.02; geometry collision cylinder length=0.020 radius=0.004; visual cylinder length=0.020 radius=0.004
- link l_pinky_proximal: mass None -> 0.055; geometry collision cylinder length=0.032 radius=0.0065; visual cylinder length=0.032 radius=0.0065
- link l_ring_distal: mass None -> 0.025; geometry collision cylinder length=0.024 radius=0.005; visual cylinder length=0.024 radius=0.005
- link l_ring_proximal: mass None -> 0.07; geometry collision cylinder length=0.038 radius=0.0075; visual cylinder length=0.038 radius=0.0075
- link l_shoulder_1: mass None -> 0.4; geometry collision sphere radius=0.04; visual mesh filename=package://humanoid_robot/meshes/l_shoulder_1.dae scale=0.001 0.001 0.001
- link l_shoulder_2: mass None -> 0.35; geometry collision sphere radius=0.035; visual mesh filename=package://humanoid_robot/meshes/l_shoulder_2.dae scale=0.001 0.001 0.001
- link l_shoulder_3: mass None -> 0.3; geometry collision sphere radius=0.03; visual mesh filename=package://humanoid_robot/meshes/l_shoulder_3.dae scale=0.001 0.001 0.001
- link l_sole: mass None -> 0.1
- link l_thumb_distal: mass None -> 0.05; geometry collision cylinder length=0.027 radius=0.007; visual cylinder length=0.027 radius=0.007
- link l_thumb_proximal: mass None -> 0.10; geometry collision cylinder length=0.038 radius=0.009; visual cylinder length=0.038 radius=0.009
- link l_upper_arm: mass None -> 0.35; geometry collision cylinder length=0.2 radius=0.025; visual mesh filename=package://humanoid_robot/meshes/l_upper_arm.dae scale=0.001 0.001 0.001
- link l_upper_leg: mass None -> 0.6; geometry collision cylinder length=0.25 radius=0.035; visual mesh filename=package://humanoid_robot/meshes/l_upper_leg.dae scale=0.001 0.001 0.001
- link l_wrist_1: mass None -> 0.15; geometry collision sphere radius=0.02; visual mesh filename=package://humanoid_robot/meshes/l_wrist_1.dae scale=0.001 0.001 0.001
- link neck_1: mass None -> 0.3; geometry collision sphere radius=0.03; visual mesh filename=package://humanoid_robot/meshes/neck_1.dae scale=0.001 0.001 0.001
- link neck_2: mass None -> 0.25; geometry collision sphere radius=0.025; visual mesh filename=package://humanoid_robot/meshes/neck_2.dae scale=0.001 0.001 0.001
- link r_ankle_1: mass None -> 0.3; geometry collision sphere radius=0.03; visual mesh filename=package://humanoid_robot/meshes/r_ankle_1.dae scale=0.001 0.001 0.001
- link r_ankle_2: mass None -> 0.25; geometry collision sphere radius=0.028; visual mesh filename=package://humanoid_robot/meshes/r_ankle_2.dae scale=0.001 0.001 0.001
- link r_elbow_1: mass None -> 0.25; geometry collision sphere radius=0.025; visual mesh filename=package://humanoid_robot/meshes/r_elbow_1.dae scale=0.001 0.001 0.001
- link r_eye: mass None -> 0.01
- link r_foot: mass None -> 0.4; geometry collision box size=0.1 0.08 0.02; visual mesh filename=package://humanoid_robot/meshes/r_foot.dae scale=0.001 0.001 0.001
- link r_forearm: mass None -> 0.3; geometry collision cylinder length=0.18 radius=0.02; visual mesh filename=package://humanoid_robot/meshes/r_forearm.dae scale=0.001 0.001 0.001
- link r_hand: mass None -> 0.2; geometry collision sphere radius=0.025; visual mesh filename=package://humanoid_robot/meshes/r_hand.dae scale=0.001 0.001 0.001
- link r_hip_1: mass None -> 0.5; geometry collision sphere radius=0.045; visual mesh filename=package://humanoid_robot/meshes/r_hip_1.dae scale=0.001 0.001 0.001
- link r_hip_2: mass None -> 0.45; geometry collision sphere radius=0.04; visual mesh filename=package://humanoid_robot/meshes/r_hip_2.dae scale=0.001 0.001 0.001
- link r_hip_3: mass None -> 0.35; geometry collision sphere radius=0.035; visual mesh filename=package://humanoid_robot/meshes/r_hip_3.dae scale=0.001 0.001 0.001
- link r_index_distal: mass None -> 0.03; geometry collision cylinder length=0.025 radius=0.006; visual cylinder length=0.025 radius=0.006
- link r_index_proximal: mass None -> 0.08; geometry collision cylinder length=0.040 radius=0.008; visual cylinder length=0.040 radius=0.008
- link r_lower_leg: mass None -> 0.5; geometry collision cylinder length=0.25 radius=0.03; visual mesh filename=package://humanoid_robot/meshes/r_lower_leg.dae scale=0.001 0.001 0.001
- link r_middle_distal: mass None -> 0.035; geometry collision cylinder length=0.028 radius=0.006; visual cylinder length=0.028 radius=0.006
- link r_middle_proximal: mass None -> 0.09; geometry collision cylinder length=0.042 radius=0.008; visual cylinder length=0.042 radius=0.008
- link r_pinky_distal: mass None -> 0.02; geometry collision cylinder length=0.020 radius=0.004; visual cylinder length=0.020 radius=0.004
- link r_pinky_proximal: mass None -> 0.055; geometry collision cylinder length=0.032 radius=0.0065; visual cylinder length=0.032 radius=0.0065
- link r_ring_distal: mass None -> 0.025; geometry collision cylinder length=0.024 radius=0.005; visual cylinder length=0.024 radius=0.005
- link r_ring_proximal: mass None -> 0.07; geometry collision cylinder length=0.038 radius=0.0075; visual cylinder length=0.038 radius=0.0075
- link r_shoulder_1: mass None -> 0.4; geometry collision sphere radius=0.04; visual mesh filename=package://humanoid_robot/meshes/r_shoulder_1.dae scale=0.001 0.001 0.001
- link r_shoulder_2: mass None -> 0.35; geometry collision sphere radius=0.035; visual mesh filename=package://humanoid_robot/meshes/r_shoulder_2.dae scale=0.001 0.001 0.001
- link r_shoulder_3: mass None -> 0.3; geometry collision sphere radius=0.03; visual mesh filename=package://humanoid_robot/meshes/r_shoulder_3.dae scale=0.001 0.001 0.001
- link r_sole: mass None -> 0.1
- link r_thumb_distal: mass None -> 0.05; geometry collision cylinder length=0.027 radius=0.007; visual cylinder length=0.027 radius=0.007
- link r_thumb_proximal: mass None -> 0.10; geometry collision cylinder length=0.038 radius=0.009; visual cylinder length=0.038 radius=0.009
- link r_upper_arm: mass None -> 0.35; geometry collision cylinder length=0.2 radius=0.025; visual mesh filename=package://humanoid_robot/meshes/r_upper_arm.dae scale=0.001 0.001 0.001
- link r_upper_leg: mass None -> 0.6; geometry collision cylinder length=0.25 radius=0.035; visual mesh filename=package://humanoid_robot/meshes/r_upper_leg.dae scale=0.001 0.001 0.001
- link r_wrist_1: mass None -> 0.15; geometry collision sphere radius=0.02; visual mesh filename=package://humanoid_robot/meshes/r_wrist_1.dae scale=0.001 0.001 0.001
- link root_link: mass None -> 1.0; geometry collision mesh filename=package://humanoid_robot/meshes/root.dae scale=0.001 0.001 0.001; visual mesh filename=package://humanoid_robot/meshes/root.dae scale=0.001 0.001 0.001
- link torso_1: mass None -> 0.8; geometry collision sphere radius=0.08; visual mesh filename=package://humanoid_robot/meshes/torso_1.dae scale=0.001 0.001 0.001
- link torso_2: mass None -> 0.7; geometry collision sphere radius=0.08; visual mesh filename=package://humanoid_robot/meshes/torso_2.dae scale=0.001 0.001 0.001
Joints:
- removed joint l_index_distal_j
- removed joint l_index_proximal_j
- removed joint l_middle_distal_j
- removed joint l_middle_proximal_j
- removed joint l_pinky_distal_j
- removed joint l_pinky_proximal_j
- removed joint l_ring_distal_j
- removed joint l_ring_proximal_j
- removed joint l_thumb_distal_j
- removed joint l_thumb_proximal_j
- removed joint r_index_distal_j
- removed joint r_index_proximal_j
- removed joint r_middle_distal_j
- removed joint r_middle_proximal_j
- removed joint r_pinky_distal_j
- removed joint r_pinky_proximal_j
- removed joint r_ring_distal_j
- removed joint r_ring_proximal_j
- removed joint r_thumb_distal_j
- removed joint r_thumb_proximal_j
- added joint l_index_distal_joint: type revolute, parent l_index_middle, child l_index_distal, origin xyz=0 0 -0.030 rpy=0 0 0, axis 0 -1 0, limit lower=-0.349066 upper=0.785398 effort=5 velocity=2.0
- added joint l_index_middle_joint: type revolute, parent l_index_proximal, child l_index_middle, origin xyz=0 0 -0.040 rpy=0 0 0, axis 0 -1 0, limit lower=-0.698132 upper=1.396263 effort=8 velocity=2.0
- added joint l_index_proximal_joint: type revolute, parent l_hand, child l_index_proximal, origin xyz=0.012 0.02 -0.075 rpy=0 0 0, axis 0 -1 0, limit lower=-0.785398 upper=1.570796 effort=10 velocity=2.0
- added joint l_middle_distal_joint: type revolute, parent l_middle_middle, child l_middle_distal, origin xyz=0 0 -0.034 rpy=0 0 0, axis 0 -1 0, limit lower=-0.349066 upper=0.785398 effort=5 velocity=2.0
- added joint l_middle_middle_joint: type revolute, parent l_middle_proximal, child l_middle_middle, origin xyz=0 0 -0.042 rpy=0 0 0, axis 0 -1 0, limit lower=-0.698132 upper=1.396263 effort=8 velocity=2.0
- added joint l_middle_proximal_joint: type revolute, parent l_hand, child l_middle_proximal, origin xyz=0.004 0.02 -0.075 rpy=0 0 0, axis 0 -1 0, limit lower=-0.785398 upper=1.570796 effort=10 velocity=2.0
- added joint l_pinky_distal_joint: type revolute, parent l_pinky_middle, child l_pinky_distal, origin xyz=0 0 -0.024 rpy=0 0 0, axis 0 -1 0, limit lower=-0.349066 upper=0.785398 effort=4 velocity=2.0
- added joint l_pinky_middle_joint: type revolute, parent l_pinky_proximal, child l_pinky_middle, origin xyz=0 0 -0.032 rpy=0 0 0, axis 0 -1 0, limit lower=-0.698132 upper=1.396263 effort=6 velocity=2.0
- added joint l_pinky_proximal_joint: type revolute, parent l_hand, child l_pinky_proximal, origin xyz=-0.012 0.018 -0.065 rpy=0 0 0, axis 0 -1 0, limit lower=-0.785398 upper=1.570796 effort=8 velocity=2.0
- added joint l_ring_distal_joint: type revolute, parent l_ring_middle, child l_ring_distal, origin xyz=0 0 -0.028 rpy=0 0 0, axis 0 -1 0, limit lower=-0.349066 upper=0.785398 effort=5 velocity=2.0
- added joint l_ring_middle_joint: type revolute, parent l_ring_proximal, child l_ring_middle, origin xyz=0 0 -0.038 rpy=0 0 0, axis 0 -1 0, limit lower=-0.698132 upper=1.396263 effort=7 velocity=2.0
- added joint l_ring_proximal_joint: type revolute, parent l_hand, child l_ring_proximal, origin xyz=-0.004 0.02 -0.073 rpy=0 0 0, axis 0 -1 0, limit lower=-0.785398 upper=1.570796 effort=9 velocity=2.0
- added joint l_thumb_distal_joint: type revolute, parent l_thumb_middle, child l_thumb_distal, origin xyz=0 0 -0.032 rpy=0 0 0, axis 0 -1 0, limit lower=-0.349066 upper=0.785398 effort=6 velocity=2.0
- added joint l_thumb_middle_joint: type revolute, parent l_thumb_proximal, child l_thumb_middle, origin xyz=0 0 -0.038 rpy=0 0 0, axis 0 -1 0, limit lower=-0.698132 upper=1.396263 effort=9 velocity=2.0
- added joint l_thumb_proximal_joint: type revolute, parent l_hand, child l_thumb_proximal, origin xyz=0.025 0.005 -0.040 rpy=0 0.5 0, axis 1 0 0, limit lower=-0.785398 upper=1.047198 effort=12 velocity=2.0
- added joint r_index_distal_joint: type revolute, parent r_index_middle, child r_index_distal, origin xyz=0 0 -0.030 rpy=0 0 0, axis 0 1 0, limit lower=-0.349066 upper=0.785398 effort=5 velocity=2.0
- added joint r_index_middle_joint: type revolute, parent r_index_proximal, child r_index_middle, origin xyz=0 0 -0.040 rpy=0 0 0, axis 0 1 0, limit lower=-0.698132 upper=1.396263 effort=8 velocity=2.0
- added joint r_index_proximal_joint: type revolute, parent r_hand, child r_index_proximal, origin xyz=-0.012 0.02 -0.075 rpy=0 0 0, axis 0 1 0, limit lower=-0.785398 upper=1.570796 effort=10 velocity=2.0
- added joint r_middle_distal_joint: type revolute, parent r_middle_middle, child r_middle_distal, origin xyz=0 0 -0.034 rpy=0 0 0, axis 0 1 0, limit lower=-0.349066 upper=0.785398 effort=5 velocity=2.0
- added joint r_middle_middle_joint: type revolute, parent r_middle_proximal, child r_middle_middle, origin xyz=0 0 -0.042 rpy=0 0 0, axis 0 1 0, limit lower=-0.698132 upper=1.396263 effort=8 velocity=2.0
- added joint r_middle_proximal_joint: type revolute, parent r_hand, child r_middle_proximal, origin xyz=-0.004 0.02 -0.075 rpy=0 0 0, axis 0 1 0, limit lower=-0.785398 upper=1.570796 effort=10 velocity=2.0
- added joint r_pinky_distal_joint: type revolute, parent r_pinky_middle, child r_pinky_distal, origin xyz=0 0 -0.024 rpy=0 0 0, axis 0 1 0, limit lower=-0.349066 upper=0.785398 effort=4 velocity=2.0
- added joint r_pinky_middle_joint: type revolute, parent r_pinky_proximal, child r_pinky_middle, origin xyz=0 0 -0.032 rpy=0 0 0, axis 0 1 0, limit lower=-0.698132 upper=1.396263 effort=6 velocity=2.0
- added joint r_pinky_proximal_joint: type revolute, parent r_hand, child r_pinky_proximal, origin xyz=0.012 0.018 -0.065 rpy=0 0 0, axis 0 1 0, limit lower=-0.785398 upper=1.570796 effort=8 velocity=2.0
- added joint r_ring_distal_joint: type revolute, parent r_ring_middle, child r_ring_distal, origin xyz=0 0 -0.028 rpy=0 0 0, axis 0 1 0, limit lower=-0.349066 upper=0.785398 effort=5 velocity=2.0
- added joint r_ring_middle_joint: type revolute, parent r_ring_proximal, child r_ring_middle, origin xyz=0 0 -0.038 rpy=0 0 0, axis 0 1 0, limit lower=-0.698132 upper=1.396263 effort=7 velocity=2.0
- added joint r_ring_proximal_joint: type revolute, parent r_hand, child r_ring_proximal, origin xyz=0.004 0.02 -0.073 rpy=0 0 0, axis 0 1 0, limit lower=-0.785398 upper=1.570796 effort=9 velocity=2.0
- added joint r_thumb_distal_joint: type revolute, parent r_thumb_middle, child r_thumb_distal, origin xyz=0 0 -0.032 rpy=0 0 0, axis 0 -1 0, limit lower=-0.349066 upper=0.785398 effort=6 velocity=2.0
- added joint r_thumb_middle_joint: type revolute, parent r_thumb_proximal, child r_thumb_middle, origin xyz=0 0 -0.038 rpy=0 0 0, axis 0 -1 0, limit lower=-0.698132 upper=1.396263 effort=9 velocity=2.0
- added joint r_thumb_proximal_joint: type revolute, parent r_hand, child r_thumb_proximal, origin xyz=-0.025 0.005 -0.040 rpy=0 -0.5 0, axis -1 0 0, limit lower=-0.785398 upper=1.047198 effort=12 velocity=2.0
